File: hw/usbavrfloppy.sch (KiCad schematic (older format))
At the start: 20 parts, among them CON1 avr_isp, J1 bothdrv, J2 floppy_conn, J3 floppy_power, J4 usbpower, J5 USB_B, J6 PWRIN, J7 USB_OTG, U1 ATMEGA88A-PU, U2 FT232RL, Y1 16MHz

Commit message: Inserted New Design Files
Parts:
- removed CON1: avr_isp, Connectors:IDC_Header_Straight_6pins, symbol avr_isp
- removed J4: usbpower, Pin_Headers:Pin_Header_Straight_1x02_Pitch2.54mm, symbol CONN_01X02
- removed U1: ATMEGA88A-PU, Housings_DIP:DIP-28_W7.62mm_Socket, symbol ATMEGA88A-PU
- added CON1: CONN_02X03, Pin_Headers:Pin_Header_Angled_2x03, symbol CONN_02X03
- added D2, D3: Led_Small, LEDs:LED_0805, symbol Led_Small
- added P1: CONN_01X03, Pin_Headers:Pin_Header_Straight_1x03, symbol CONN_01X03
- added P2, P3, P4, P5: CONN_01X01, Connect:1pin, symbol CONN_01X01
- added Q1, Q10, Q2, Q3, Q4, Q5, Q6, Q7, Q8, Q9: BSS138, TO_SOT_Packages_SMD:SOT-23, symbol BSS138
- added R10, R11, R12, R13, R14, R15, R16, R17, R18, R19, R20, R21, R24, R25, R26, R3, R4, R5, R6, R7, R8, R9: 10k, Resistors_SMD:R_0805_HandSoldering, symbol R
- added R22: 1k, Resistors_SMD:R_0805_HandSoldering, symbol R
- added R23: 330, Resistors_SMD:R_0805_HandSoldering, symbol R
- added R27: 4.7k, Resistors_SMD:R_0805_HandSoldering, symbol R
- added SW1: ~mRESET, Buttons_Switches_SMD:SW_SPST_FSMSM, symbol SW_PUSH
- added U1: ATMEGA88-A, Housings_QFP:TQFP-32_7x7mm_Pitch0.8mm, symbol ATMEGA88-A
- C3, C4, C6: value 0.1uF -> 100nF
- C5: footprint Capacitors_SMD:CP_Elec_5x5.7 -> Capacitors_SMD:c_elec_5x5.7
- D1: symbol LED_Small -> Led_Small
- J1: footprint Pin_Headers:Pin_Header_Straight_1x02_Pitch2.54mm -> Pin_Headers:Pin_Header_Straight_1x02
- J2: footprint Connectors:IDC_Header_Straight_34pins -> Connect:IDC_Header_Straight_34pins
- J3: footprint Connectors_Molex:Molex_KK-6410-04_04x2.54mm_Straight -> Pin_Headers:Pin_Header_Straight_1x04
- J5: footprint Connectors:USB_B -> RetroBitLab:USB_Mini-B_Large_Pads
- J6: footprint Connectors_Molex:Molex_SPOX-5267_22-03-5045_04x2.54mm_Straight -> Pin_Headers:Pin_Header_Angled_1x04
- J7: footprint Connectors:USB_Mini-B -> RetroBitLab:USB_Micro-B_Large_Pads
- R2: value 1k -> 10k
- U2: symbol FT232RL -> FT232RL-RESCUE-usbavrfloppy
- Y1: footprint Crystals:Crystal_SMD_HC49-SD -> Crystals:Crystal_HC49-SD_SMD
Connections:
- net labels added: VCC_USB, Vcc_FLOPPY, Vcc_MCU, ~MOTEB, ~SIDE1, ~WPROT, ~mDIR, ~mHSEL, ~mINDEX, ~mMOTEN, ~mRDATA, ~mRESET, ~mSTEP, ~mTRK0, ~mWDATA, ~mWGATE, ~mWPROTECT
- net labels removed: ~HSEL, ~MOTEN, ~RESET, ~WPROTECT
- wire segments 93 -> 113
- no-connect marks 21 -> 27
Other:
- note added: "MOUNTING HOLES"
- note added: "Need to be replaced if SoC is not 5V tolerant"

Commit message: Re-generated after libraries cleanup
Parts:
- removed U2: FT232RL, Housings_SSOP:SSOP-28_5.3x10.2mm_Pitch0.65mm, symbol FT232RL-RESCUE-usbavrfloppy
- added U2: FT232RL, Housings_SSOP:SSOP-28_5.3x10.2mm_Pitch0.65mm, symbol FT232RL
- J2: symbol floppy_conn -> CONN_02X17
Connections:
- no-connect marks 27 -> 29
Changed lines of the file:
@@
 EESchema Schematic File Version 2
-LIBS:usbavrfloppy-rescue
 LIBS:power
 LIBS:device
@@
 LIBS:valves
 LIBS:ftdi
-LIBS:usbavrfloppy
 LIBS:switches
-LIBS:usbavrfloppy-cache
 EELAYER 25 0
 EELAYER END
@@
 encoding utf-8
 Sheet 1 1
-Title "USB amiga floppy controller"
+Title "USB AVR Amiga Floppy Controller"
 Date "2018-03-01"
 Rev "1"
-Comp ""
+Comp "RetroBit Lab"
 Comment1 "Creative Commons Attribution Share-Alike (CC BY-SA)"
 Comment2 "Original Concepts Copyright (C) John Tsiombikas 2018"
@@
 $EndDescr
 $Comp
-L floppy_conn J2
+L CONN_02X17 J2
 U 1 1 5A96F2AA
-P 9850 2200
-F 0 "J2" H 9850 3100 50  0000 C CNN
-F 1 "floppy_conn" V 9850 2200 50  0000 C CNN
-F 2 "Connect:IDC_Header_Straight_34pins" H 9850 1100 50  0001 C CNN
-F 3 "" H 9850 1100 50  0001 C CNN
-	1    9850 2200
+P 10050 2200
+F 0 "J2" H 10050 3100 50  0000 C CNN
+F 1 "floppy_conn" V 10050 2200 50  0000 C CNN
+F 2 "Connect:IDC_Header_Straight_34pins" H 10050 1100 50  0001 C CNN
+F 3 "" H 10050 1100 50  0001 C CNN
+	1    10050 2200
 	-1   0    0    -1
 $EndComp
@@
 L CONN_01X02 J1
 U 1 1 5A96F78C
-P 8900 1600
-F 0 "J1" H 8900 1750 50  0000 C CNN
-F 1 "bothdrv" V 9000 1600 50  0000 C CNN
-F 2 "Pin_Headers:Pin_Header_Straight_1x02" H 8900 1600 50  0001 C CNN
-F 3 "" H 8900 1600 50  0001 C CNN
-	1    8900 1600
+P 9300 1600
+F 0 "J1" H 9300 1750 50  0000 C CNN
+F 1 "bothdrv" V 9400 1600 50  0000 C CNN
+F 2 "Pin_Headers:Pin_Header_Straight_1x02" H 9300 1600 50  0001 C CNN
+F 3 "" H 9300 1600 50  0001 C CNN
+	1    9300 1600
 	0    -1   -1   0
 $EndComp
@@
 Text Label 3900 1300 0    60   ~ 0
 ~mHSEL
-NoConn ~ 9400 3000
-NoConn ~ 9400 1400
+NoConn ~ 9800 3000
+NoConn ~ 9800 1400
 Text Label 3900 3000 0    60   ~ 0
 ~mINDEX
@@
 L GND #PWR03
 U 1 1 5A971B5E
-P 3150 6100
-F 0 "#PWR03" H 3150 5850 50  0001 C CNN
-F 1 "GND" H 3150 5950 39  0000 C CNN
-F 2 "" H 3150 6100 50  0001 C CNN
-F 3 "" H 3150 6100 50  0001 C CNN
-	1    3150 6100
+P 3250 6100
+F 0 "#PWR03" H 3250 5850 50  0001 C CNN
+F 1 "GND" H 3250 5950 39  0000 C CNN
+F 2 "" H 3250 6100 50  0001 C CNN
+F 3 "" H 3250 6100 50  0001 C CNN
+	1    3250 6100
 	1    0    0    -1
 $EndComp
@@
 Connection ~ 10200 4550
 Wire Wire Line
-	8950 1800 9400 1800
-Wire Wire Line
-	9400 2000 9250 2000
-Wire Wire Line
-	9250 2000 9250 1800
-Connection ~ 9250 1800
-Wire Wire Line
-	8850 1900 9400 1900
-Wire Wire Line
-	9200 2100 9200 1900
-Connection ~ 9200 1900
+	9350 1800 9800 1800
+Wire Wire Line
+	9800 2000 9650 2000
+Wire Wire Line
+	9650 2000 9650 1800
+Connection ~ 9650 1800
+Wire Wire Line
+	9250 1900 9800 1900
+Wire Wire Line
+	9600 2100 9600 1900
+Connection ~ 9600 1900
 Wire Wire Line
 	3900 2900 4600 2900
@@
 	4700 4400 4250 4400
 Wire Wire Line
-	4250 4700 4500 4700
-Wire Wire Line
-	4500 4700 4500 2250
-Connection ~ 3600 4100
+	4500 4700 4250 4700
+Wire Wire Line
+	4500 2250 4500 4700
 Wire Wire Line
 	2550 4400 2650 4400
@@
 Connection ~ 10300 2900
 Connection ~ 10300 3000
-Connection ~ 9200 2100
+Connection ~ 9600 2100
 Wire Wire Line
 	4200 1700 4200 1450
@@
 Text Label 4050 7150 2    60   ~ 0
 ~mSTEP
-Text Label 9400 2600 2    60   ~ 0
+Text Label 9800 2600 2    60   ~ 0
 ~TRK0
 Text Label 6400 1450 0    60   ~ 0
 ~TRK0
-Text Label 9400 2900 2    60   ~ 0
+Text Label 9800 2900 2    60   ~ 0
 ~SIDE1
 Text Label 8250 1450 0    60   ~ 0
 ~SIDE1
-Text Label 9400 2500 2    60   ~ 0
+Text Label 9800 2500 2    60   ~ 0
 ~WGATE
 Text Label 6400 2800 0    60   ~ 0
@@
 Text Label 8300 2800 0    60   ~ 0
 ~WPROT
-Text Label 9400 2700 2    60   ~ 0
+Text Label 9800 2700 2    60   ~ 0
 ~WPROT
-Text Label 9400 1700 2    60   ~ 0
+Text Label 9800 1700 2    60   ~ 0
 ~INDEX
 Wire Wire Line
-	9000 2100 9400 2100
-Wire Wire Line
-	8850 1900 8850 1800
+	9400 2100 9800 2100
+Wire Wire Line
+	9250 1900 9250 1800
 Text Label 6400 4150 0    60   ~ 0
 ~INDEX
-Text Label 9400 2400 2    60   ~ 0
+Text Label 9800 2400 2    60   ~ 0
 ~WDATA
 Text Label 8200 4150 0    60   ~ 0
 ~WDATA
-Text Label 9400 2800 2    60   ~ 0
+Text Label 9800 2800 2    60   ~ 0
 ~RDATA
 Text Label 6400 5500 0    60   ~ 0
 ~RDATA
-Text Label 9000 2100 2    60   ~ 0
+Text Label 9400 2100 2    60   ~ 0
 ~MOTEB
 Text Label 8250 5500 0    60   ~ 0
@@
 Text Label 6400 7150 0    60   ~ 0
 ~DIR
-Text Label 9400 2200 2    60   ~ 0
+Text Label 9800 2200 2    60   ~ 0
 ~DIR
 Text Label 4900 7150 0    60   ~ 0
 ~STEP
-Text Label 9400 2300 2    60   ~ 0
+Text Label 9800 2300 2    60   ~ 0
 ~STEP
 Text GLabel 2000 1000 1    60   Input ~ 0
@@
 Connection ~ 4750 1600
 Wire Wire Line
-	1450 2950 950  2950
+	950  2950 1450 2950
 Wire Wire Line
 	1200 2950 1200 2850
@@
 Wire Wire Line
 	10600 5500 10600 5650
-Connection ~ 10300 3050
 Wire Wire Line
 	950  3250 1450 3250
@@
 Text GLabel 1100 1950 0    60   Input ~ 0
 VCC_USB
-$Comp
-L FT232RL-RESCUE-usbavrfloppy U2
-U 1 1 5A95DEF7
-P 3450 5100
-F 0 "U2" H 2800 6000 50  0000 L CNN
-F 1 "FT232RL" H 3850 6000 50  0000 L CNN
-F 2 "Housings_SSOP:SSOP-28_5.3x10.2mm_Pitch0.65mm" H 3450 5100 50  0001 C CNN
-F 3 "" H 3450 5100 50  0001 C CNN
-	1    3450 5100
-	1    0    0    -1
-$EndComp
 Text GLabel 2650 5800 0    60   Input ~ 0
 GND
@@
 L GND #PWR031
 U 1 1 5BE7A7E8
-P 3350 6100
-F 0 "#PWR031" H 3350 5850 50  0001 C CNN
-F 1 "GND" H 3350 5950 39  0000 C CNN
-F 2 "" H 3350 6100 50  0001 C CNN
-F 3 "" H 3350 6100 50  0001 C CNN
-	1    3350 6100
+P 3450 6100
+F 0 "#PWR031" H 3450 5850 50  0001 C CNN
+F 1 "GND" H 3450 5950 39  0000 C CNN
+F 2 "" H 3450 6100 50  0001 C CNN
+F 3 "" H 3450 6100 50  0001 C CNN
+	1    3450 6100
 	1    0    0    -1
 $EndComp
@@
 L GND #PWR033
 U 1 1 5BE7A95A
-P 3750 6100
-F 0 "#PWR033" H 3750 5850 50  0001 C CNN
-F 1 "GND" H 3750 5950 39  0000 C CNN
-F 2 "" H 3750 6100 50  0001 C CNN
-F 3 "" H 3750 6100 50  0001 C CNN
-	1    3750 6100
-	1    0    0    -1
-$EndComp
-Wire Wire Line
-	3400 4100 3600 4100
-Wire Wire Line
-	3650 3950 3600 3950
-Wire Wire Line
-	3600 3950 3600 4100
+P 3650 6100
+F 0 "#PWR033" H 3650 5850 50  0001 C CNN
+F 1 "GND" H 3650 5950 39  0000 C CNN
+F 2 "" H 3650 6100 50  0001 C CNN
+F 3 "" H 3650 6100 50  0001 C CNN
+	1    3650 6100
+	1    0    0    -1
+$EndComp
+Wire Wire Line
+	3550 3950 3650 3950
 Text GLabel 1300 4050 2    60   Input ~ 0
 Vcc_MCU
@@
 Text Notes 600  5200 1    60   Italic 0
 Need to be replaced if SoC is not 5V tolerant
+$Comp
+L FT232RL U2
+U 1 1 5C1FFB63
+P 3450 5100
+F 0 "U2" H 2800 6000 50  0000 L CNN
+F 1 "FT232RL" H 3850 6000 50  0000 L CNN
+F 2 "Housings_SSOP:SSOP-28_5.3x10.2mm_Pitch0.65mm" H 3450 5100 50  0001 C CNN
+F 3 "" H 3450 5100 50  0000 C CNN
+	1    3450 5100
+	1    0    0    -1
+$EndComp
+Wire Wire Line
+	3550 4100 3350 4100
+Wire Wire Line
+	3550 3950 3550 4100
+Connection ~ 3550 4100
+NoConn ~ 9800 1500
+NoConn ~ 9800 1600
 $EndSCHEMATC

Commit message: Modified for new 3d components and logos
Parts:
- SW1: footprint Buttons_Switches_SMD:SW_SPST_FSMSM -> RetroBitLab:SW_SPST_FSMSM_3D
Changed lines of the file:
@@
 LIBS:ftdi
 LIBS:switches
+LIBS:AmigaComponents
+LIBS:4xxx
+LIBS:4xxx_IEEE
+LIBS:74xGxx
+LIBS:74xx_IEEE
+LIBS:Amplifier_Audio
+LIBS:Amplifier_Buffer
+LIBS:Amplifier_Current
+LIBS:Amplifier_Difference
+LIBS:Amplifier_Instrumentation
+LIBS:Amplifier_Operational
+LIBS:Amplifier_Video
+LIBS:Analog
+LIBS:Analog_ADC
+LIBS:Analog_DAC
+LIBS:Analog_Switch
+LIBS:Audio
+LIBS:Battery_Management
+LIBS:Comparator
+LIBS:Connector
+LIBS:Connector_Generic
+LIBS:Connector_Generic_MountingPin
+LIBS:Connector_Generic_Shielded
+LIBS:Converter_ACDC
+LIBS:Converter_DCDC
+LIBS:CPLD_Altera
+LIBS:CPLD_Xilinx
+LIBS:CPU
+LIBS:CPU_NXP_6800
+LIBS:CPU_NXP_68000
+LIBS:CPU_PowerPC
+LIBS:Device
+LIBS:Diode
+LIBS:Diode_Bridge
+LIBS:Diode_Laser
+LIBS:Display_Character
+LIBS:Display_Graphic
+LIBS:Driver_Display
+LIBS:Driver_FET
+LIBS:Driver_LED
+LIBS:Driver_Motor
+LIBS:Driver_Relay
+LIBS:DSP_AnalogDevices
+LIBS:DSP_Freescale
+LIBS:DSP_Microchip_DSPIC33
+LIBS:DSP_Motorola
+LIBS:DSP_Texas
+LIBS:Fiber_Optic
+LIBS:Filter
+LIBS:FPGA_Lattice
+LIBS:FPGA_Microsemi
+LIBS:FPGA_Xilinx
+LIBS:FPGA_Xilinx_Artix7
+LIBS:FPGA_Xilinx_Kintex7
+LIBS:FPGA_Xilinx_Spartan6
+LIBS:FPGA_Xilinx_Virtex5
+LIBS:FPGA_Xilinx_Virtex6
+LIBS:FPGA_Xilinx_Virtex7
+LIBS:ft232rl
+LIBS:GPU
+LIBS:Graphic
+LIBS:Interface
+LIBS:Interface_CAN_LIN
+LIBS:Interface_CurrentLoop
+LIBS:Interface_Ethernet
+LIBS:Interface_Expansion
+LIBS:Interface_HID
+LIBS:Interface_LineDriver
+LIBS:Interface_Optical
+LIBS:Interface_Telecom
+LIBS:Interface_UART
+LIBS:Interface_USB
+LIBS:Isolator
+LIBS:Isolator_Analog
+LIBS:Jumper
+LIBS:LED
+LIBS:Logic_LevelTranslator
+LIBS:Logic_Programmable
+LIBS:MCU_AnalogDevices
+LIBS:MCU_Cypress
+LIBS:MCU_Espressif
+LIBS:MCU_Intel
+LIBS:MCU_Microchip_8051
+LIBS:MCU_Microchip_ATmega
+LIBS:MCU_Microchip_ATtiny
+LIBS:MCU_Microchip_AVR
+LIBS:MCU_Microchip_PIC10
+LIBS:MCU_Microchip_PIC12
+LIBS:MCU_Microchip_PIC16
+LIBS:MCU_Microchip_PIC18
+LIBS:MCU_Microchip_PIC24
+LIBS:MCU_Microchip_PIC32
+LIBS:MCU_Microchip_SAMD
+LIBS:MCU_Microchip_SAME
+LIBS:MCU_Microchip_SAML
+LIBS:MCU_Module
+LIBS:MCU_Nordic
+LIBS:MCU_NXP_ColdFire
+LIBS:MCU_NXP_HC11
+LIBS:MCU_NXP_HC12
+LIBS:MCU_NXP_HCS12
+LIBS:MCU_NXP_Kinetis
+LIBS:MCU_NXP_LPC
+LIBS:MCU_NXP_MAC7100
+LIBS:MCU_NXP_MCore
+LIBS:MCU_NXP_S08
+LIBS:MCU_Parallax
+LIBS:MCU_SiFive
+LIBS:MCU_SiliconLabs
+LIBS:MCU_ST_STM8
+LIBS:MCU_ST_STM32F0
+LIBS:MCU_ST_STM32F1
+LIBS:MCU_ST_STM32F2
+LIBS:MCU_ST_STM32F3
+LIBS:MCU_ST_STM32F4
+LIBS:MCU_ST_STM32F7
+LIBS:MCU_ST_STM32H7
+LIBS:MCU_ST_STM32L0
+LIBS:MCU_ST_STM32L1
+LIBS:MCU_ST_STM32L4
+LIBS:MCU_ST_STM32L4+
+LIBS:MCU_Texas
+LIBS:MCU_Texas_MSP430
+LIBS:Mechanical
+LIBS:Memory_Controller
+LIBS:Memory_EEPROM
+LIBS:Memory_EPROM
+LIBS:Memory_Flash
+LIBS:Memory_NVRAM
+LIBS:Memory_RAM
+LIBS:Memory_ROM
+LIBS:Memory_UniqueID
+LIBS:Motor
+LIBS:Oscillator
+LIBS:Potentiometer_Digital
+LIBS:Power_Management
+LIBS:Power_Protection
+LIBS:Power_Supervisor
+LIBS:pspice
+LIBS:Reference_Current
+LIBS:Reference_Voltage
+LIBS:Regulator_Controller
+LIBS:Regulator_Current
+LIBS:Regulator_Linear
+LIBS:Regulator_SwitchedCapacitor
+LIBS:Regulator_Switching
+LIBS:Relay
+LIBS:Relay_SolidState
+LIBS:RF
+LIBS:RF_AM_FM
+LIBS:RF_Amplifier
+LIBS:RF_Bluetooth
+LIBS:RF_GPS
+LIBS:RF_GSM
+LIBS:RF_Mixer
+LIBS:RF_Module
+LIBS:RF_RFID
+LIBS:RF_Switch
+LIBS:RF_WiFi
+LIBS:RF_ZigBee
+LIBS:Security
+LIBS:Sensor
+LIBS:Sensor_Audio
+LIBS:Sensor_Current
+LIBS:Sensor_Gas
+LIBS:Sensor_Humidity
+LIBS:Sensor_Magnetic
+LIBS:Sensor_Motion
+LIBS:Sensor_Optical
+LIBS:Sensor_Pressure
+LIBS:Sensor_Proximity
+LIBS:Sensor_Temperature
+LIBS:Sensor_Touch
+LIBS:Sensor_Voltage
+LIBS:Switch
+LIBS:Timer
+LIBS:Timer_PLL
+LIBS:Timer_RTC
+LIBS:Transformer
+LIBS:Transistor_Array
+LIBS:Transistor_BJT
+LIBS:Transistor_FET
+LIBS:Transistor_IGBT
+LIBS:Triac_Thyristor
+LIBS:Valve
+LIBS:Video
+LIBS:usbavrfloppy-cache
 EELAYER 25 0
 EELAYER END
@@
 F 0 "SW1" H 2150 7010 50  0000 C CNN
 F 1 "~mRESET" H 2000 6820 50  0000 C CNN
-F 2 "Buttons_Switches_SMD:SW_SPST_FSMSM" H 2000 6900 50  0001 C CNN
+F 2 "RetroBitLab:SW_SPST_FSMSM_3D" H 2000 6900 50  0001 C CNN
 F 3 "" H 2000 6900 50  0000 C CNN
 	1    2000 6900

Commit message: Added footprint for idc connector
Parts:
- J2: footprint Connect:IDC_Header_Straight_34pins -> RetroBitLab:IDC-Header_2x17_P2.54mm_Vertical_Lock
Changed lines of the file:
@@
 F 0 "J2" H 10050 3100 50  0000 C CNN
 F 1 "floppy_conn" V 10050 2200 50  0000 C CNN
-F 2 "Connect:IDC_Header_Straight_34pins" H 10050 1100 50  0001 C CNN
+F 2 "RetroBitLab:IDC-Header_2x17_P2.54mm_Vertical_Lock" H 10050 1100 50  0001 C CNN
 F 3 "" H 10050 1100 50  0001 C CNN
 	1    10050 2200
