File: hw/usbavrfloppy.sch (KiCad schematic (older format))
At the start: 62 parts, among them CON1 CONN_02X03, J1 bothdrv, J2 floppy_conn, J3 floppy_power, J5 USB_B, J6 PWRIN, J7 USB_OTG, P1 CONN_01X03, P2 CONN_01X01, P3 CONN_01X01, P4 CONN_01X01, P5 CONN_01X01, Q1 BSS138, Q10 BSS138, Q2 BSS138, Q3 BSS138, Q4 BSS138, Q5 BSS138, Q6 BSS138, Q7 BSS138, Q8 BSS138, Q9 BSS138, SW1 ~mRESET, U1 ATMEGA88-A, U2 FT232RL, Y1 16MHz

Commit message: Changed from 0603/0806 to 1208
Parts:
- C1, C2, C3, C4, C6: footprint Capacitors_SMD:C_0805_HandSoldering -> Capacitors_SMD:C_1206_HandSoldering
- D1, D2, D3: footprint LEDs:LED_0805 -> LEDs:LED_1206
- R1, R10, R11, R12, R13, R14, R15, R16, R17, R18, R19, R2, R20, R21, R22, R23, R24, R25, R26, R27, R3, R4, R5, R6, R7, R8, R9: footprint Resistors_SMD:R_0805_HandSoldering -> Resistors_SMD:R_1206_HandSoldering
Changed lines of the file:
@@
 LIBS:FPGA_Xilinx_Virtex6
 LIBS:FPGA_Xilinx_Virtex7
-LIBS:ft232rl
 LIBS:GPU
 LIBS:Graphic
@@
 LIBS:MCU_Texas_MSP430
 LIBS:Mechanical
-LIBS:Memory_Controller
 LIBS:Memory_EEPROM
 LIBS:Memory_EPROM
@@
 LIBS:Valve
 LIBS:Video
-LIBS:usbavrfloppy-cache
 EELAYER 25 0
 EELAYER END
@@
 F 0 "C4" H 2425 4500 50  0000 L CNN
 F 1 "100nF" H 2425 4300 50  0000 L CNN
-F 2 "Capacitors_SMD:C_0805_HandSoldering" H 2438 4250 50  0001 C CNN
+F 2 "Capacitors_SMD:C_1206_HandSoldering" H 2438 4250 50  0001 C CNN
 F 3 "" H 2400 4400 50  0001 C CNN
 	1    2400 4400
@@
 F 0 "C6" H 1225 3200 50  0000 L CNN
 F 1 "100nF" H 1225 3000 50  0000 L CNN
-F 2 "Capacitors_SMD:C_0805_HandSoldering" H 1238 2950 50  0001 C CNN
+F 2 "Capacitors_SMD:C_1206_HandSoldering" H 1238 2950 50  0001 C CNN
 F 3 "" H 1200 3100 50  0001 C CNN
 	1    1200 3100
@@
 F 0 "C3" H 1475 3200 50  0000 L CNN
 F 1 "100nF" H 1475 3000 50  0000 L CNN
-F 2 "Capacitors_SMD:C_0805_HandSoldering" H 1488 2950 50  0001 C CNN
+F 2 "Capacitors_SMD:C_1206_HandSoldering" H 1488 2950 50  0001 C CNN
 F 3 "" H 1450 3100 50  0001 C CNN
 	1    1450 3100
@@
 F 0 "R1" V 4830 1450 50  0000 C CNN
 F 1 "330" V 4750 1450 50  0000 C CNN
-F 2 "Resistors_SMD:R_0805_HandSoldering" V 4680 1450 50  0001 C CNN
+F 2 "Resistors_SMD:R_1206_HandSoldering" V 4680 1450 50  0001 C CNN
 F 3 "" H 4750 1450 50  0001 C CNN
 	1    4750 1450
@@
 F 0 "D1" H 4250 1500 50  0000 L CNN
 F 1 "ACT" H 4450 1500 50  0000 L CNN
-F 2 "LEDs:LED_0805" V 4400 1450 50  0001 C CNN
+F 2 "LEDs:LED_1206" V 4400 1450 50  0001 C CNN
 F 3 "" V 4400 1450 50  0001 C CNN
 	1    4400 1450
@@
 F 0 "C2" H 4660 1970 50  0000 L CNN
 F 1 "22pF" V 4700 1650 50  0000 L CNN
-F 2 "Capacitors_SMD:C_0805_HandSoldering" H 4650 1900 50  0001 C CNN
+F 2 "Capacitors_SMD:C_1206_HandSoldering" H 4650 1900 50  0001 C CNN
 F 3 "" H 4650 1900 50  0001 C CNN
 	1    4650 1900
@@
 F 0 "C1" H 4660 1670 50  0000 L CNN
 F 1 "22pF" V 4600 1350 50  0000 L CNN
-F 2 "Capacitors_SMD:C_0805_HandSoldering" H 4650 1600 50  0001 C CNN
+F 2 "Capacitors_SMD:C_1206_HandSoldering" H 4650 1600 50  0001 C CNN
 F 3 "" H 4650 1600 50  0001 C CNN
 	1    4650 1600
@@
 F 0 "R15" V 7630 1300 50  0000 C CNN
 F 1 "10k" V 7550 1300 50  0000 C CNN
-F 2 "Resistors_SMD:R_0805_HandSoldering" V 7480 1300 50  0001 C CNN
+F 2 "Resistors_SMD:R_1206_HandSoldering" V 7480 1300 50  0001 C CNN
 F 3 "" H 7550 1300 50  0000 C CNN
 	1    7550 1300
@@
 F 0 "R19" V 8180 1300 50  0000 C CNN
 F 1 "10k" V 8100 1300 50  0000 C CNN
-F 2 "Resistors_SMD:R_0805_HandSoldering" V 8030 1300 50  0001 C CNN
+F 2 "Resistors_SMD:R_1206_HandSoldering" V 8030 1300 50  0001 C CNN
 F 3 "" H 8100 1300 50  0000 C CNN
 	1    8100 1300
@@
 F 0 "R4" V 5780 1300 50  0000 C CNN
 F 1 "10k" V 5700 1300 50  0000 C CNN
-F 2 "Resistors_SMD:R_0805_HandSoldering" V 5630 1300 50  0001 C CNN
+F 2 "Resistors_SMD:R_1206_HandSoldering" V 5630 1300 50  0001 C CNN
 F 3 "" H 5700 1300 50  0000 C CNN
 	1    5700 1300
@@
 F 0 "R9" V 6330 1300 50  0000 C CNN
 F 1 "10k" V 6250 1300 50  0000 C CNN
-F 2 "Resistors_SMD:R_0805_HandSoldering" V 6180 1300 50  0001 C CNN
+F 2 "Resistors_SMD:R_1206_HandSoldering" V 6180 1300 50  0001 C CNN
 F 3 "" H 6250 1300 50  0000 C CNN
 	1    6250 1300
@@
 F 0 "R5" V 5780 2650 50  0000 C CNN
 F 1 "10k" V 5700 2650 50  0000 C CNN
-F 2 "Resistors_SMD:R_0805_HandSoldering" V 5630 2650 50  0001 C CNN
+F 2 "Resistors_SMD:R_1206_HandSoldering" V 5630 2650 50  0001 C CNN
 F 3 "" H 5700 2650 50  0000 C CNN
 	1    5700 2650
@@
 F 0 "R10" V 6330 2650 50  0000 C CNN
 F 1 "10k" V 6250 2650 50  0000 C CNN
-F 2 "Resistors_SMD:R_0805_HandSoldering" V 6180 2650 50  0001 C CNN
+F 2 "Resistors_SMD:R_1206_HandSoldering" V 6180 2650 50  0001 C CNN
 F 3 "" H 6250 2650 50  0000 C CNN
 	1    6250 2650
@@
 F 0 "R17" V 7680 2650 50  0000 C CNN
 F 1 "10k" V 7600 2650 50  0000 C CNN
-F 2 "Resistors_SMD:R_0805_HandSoldering" V 7530 2650 50  0001 C CNN
+F 2 "Resistors_SMD:R_1206_HandSoldering" V 7530 2650 50  0001 C CNN
 F 3 "" H 7600 2650 50  0000 C CNN
 	1    7600 2650
@@
 F 0 "R21" V 8230 2650 50  0000 C CNN
 F 1 "10k" V 8150 2650 50  0000 C CNN
-F 2 "Resistors_SMD:R_0805_HandSoldering" V 8080 2650 50  0001 C CNN
+F 2 "Resistors_SMD:R_1206_HandSoldering" V 8080 2650 50  0001 C CNN
 F 3 "" H 8150 2650 50  0000 C CNN
 	1    8150 2650
@@
 F 0 "R14" V 7580 4000 50  0000 C CNN
 F 1 "10k" V 7500 4000 50  0000 C CNN
-F 2 "Resistors_SMD:R_0805_HandSoldering" V 7430 4000 50  0001 C CNN
+F 2 "Resistors_SMD:R_1206_HandSoldering" V 7430 4000 50  0001 C CNN
 F 3 "" H 7500 4000 50  0000 C CNN
 	1    7500 4000
@@
 F 0 "R18" V 8130 4000 50  0000 C CNN
 F 1 "10k" V 8050 4000 50  0000 C CNN
-F 2 "Resistors_SMD:R_0805_HandSoldering" V 7980 4000 50  0001 C CNN
+F 2 "Resistors_SMD:R_1206_HandSoldering" V 7980 4000 50  0001 C CNN
 F 3 "" H 8050 4000 50  0000 C CNN
 	1    8050 4000
@@
 F 0 "R6" V 5780 4000 50  0000 C CNN
 F 1 "10k" V 5700 4000 50  0000 C CNN
-F 2 "Resistors_SMD:R_0805_HandSoldering" V 5630 4000 50  0001 C CNN
+F 2 "Resistors_SMD:R_1206_HandSoldering" V 5630 4000 50  0001 C CNN
 F 3 "" H 5700 4000 50  0000 C CNN
 	1    5700 4000
@@
 F 0 "R11" V 6330 4000 50  0000 C CNN
 F 1 "10k" V 6250 4000 50  0000 C CNN
-F 2 "Resistors_SMD:R_0805_HandSoldering" V 6180 4000 50  0001 C CNN
+F 2 "Resistors_SMD:R_1206_HandSoldering" V 6180 4000 50  0001 C CNN
 F 3 "" H 6250 4000 50  0000 C CNN
 	1    6250 4000
@@
 F 0 "R7" V 5780 5350 50  0000 C CNN
 F 1 "10k" V 5700 5350 50  0000 C CNN
-F 2 "Resistors_SMD:R_0805_HandSoldering" V 5630 5350 50  0001 C CNN
+F 2 "Resistors_SMD:R_1206_HandSoldering" V 5630 5350 50  0001 C CNN
 F 3 "" H 5700 5350 50  0000 C CNN
 	1    5700 5350
@@
 F 0 "R12" V 6330 5350 50  0000 C CNN
 F 1 "10k" V 6250 5350 50  0000 C CNN
-F 2 "Resistors_SMD:R_0805_HandSoldering" V 6180 5350 50  0001 C CNN
+F 2 "Resistors_SMD:R_1206_HandSoldering" V 6180 5350 50  0001 C CNN
 F 3 "" H 6250 5350 50  0000 C CNN
 	1    6250 5350
@@
 F 0 "R16" V 7630 5350 50  0000 C CNN
 F 1 "10k" V 7550 5350 50  0000 C CNN
-F 2 "Resistors_SMD:R_0805_HandSoldering" V 7480 5350 50  0001 C CNN
+F 2 "Resistors_SMD:R_1206_HandSoldering" V 7480 5350 50  0001 C CNN
 F 3 "" H 7550 5350 50  0000 C CNN
 	1    7550 5350
@@
 F 0 "R20" V 8180 5350 50  0000 C CNN
 F 1 "10k" V 8100 5350 50  0000 C CNN
-F 2 "Resistors_SMD:R_0805_HandSoldering" V 8030 5350 50  0001 C CNN
+F 2 "Resistors_SMD:R_1206_HandSoldering" V 8030 5350 50  0001 C CNN
 F 3 "" H 8100 5350 50  0000 C CNN
 	1    8100 5350
@@
 F 0 "R2" V 4280 7000 50  0000 C CNN
 F 1 "10k" V 4200 7000 50  0000 C CNN
-F 2 "Resistors_SMD:R_0805_HandSoldering" V 4130 7000 50  0001 C CNN
+F 2 "Resistors_SMD:R_1206_HandSoldering" V 4130 7000 50  0001 C CNN
 F 3 "" H 4200 7000 50  0000 C CNN
 	1    4200 7000
@@
 F 0 "R3" V 4830 7000 50  0000 C CNN
 F 1 "10k" V 4750 7000 50  0000 C CNN
-F 2 "Resistors_SMD:R_0805_HandSoldering" V 4680 7000 50  0001 C CNN
+F 2 "Resistors_SMD:R_1206_HandSoldering" V 4680 7000 50  0001 C CNN
 F 3 "" H 4750 7000 50  0000 C CNN
 	1    4750 7000
@@
 F 0 "R8" V 5780 7000 50  0000 C CNN
 F 1 "10k" V 5700 7000 50  0000 C CNN
-F 2 "Resistors_SMD:R_0805_HandSoldering" V 5630 7000 50  0001 C CNN
+F 2 "Resistors_SMD:R_1206_HandSoldering" V 5630 7000 50  0001 C CNN
 F 3 "" H 5700 7000 50  0000 C CNN
 	1    5700 7000
@@
 F 0 "R13" V 6330 7000 50  0000 C CNN
 F 1 "10k" V 6250 7000 50  0000 C CNN
-F 2 "Resistors_SMD:R_0805_HandSoldering" V 6180 7000 50  0001 C CNN
+F 2 "Resistors_SMD:R_1206_HandSoldering" V 6180 7000 50  0001 C CNN
 F 3 "" H 6250 7000 50  0000 C CNN
 	1    6250 7000
@@
 F 0 "R22" V 9280 3550 50  0000 C CNN
 F 1 "1k" V 9200 3550 50  0000 C CNN
-F 2 "Resistors_SMD:R_0805_HandSoldering" V 9130 3550 50  0001 C CNN
+F 2 "Resistors_SMD:R_1206_HandSoldering" V 9130 3550 50  0001 C CNN
 F 3 "" H 9200 3550 50  0000 C CNN
 	1    9200 3550
@@
 F 0 "D2" H 9150 3925 50  0000 L CNN
 F 1 "Led_Small" H 9025 3700 50  0000 L CNN
-F 2 "LEDs:LED_0805" V 9200 3800 50  0001 C CNN
+F 2 "LEDs:LED_1206" V 9200 3800 50  0001 C CNN
 F 3 "" V 9200 3800 50  0000 C CNN
 	1    9200 3800
@@
 F 0 "R23" V 9280 4900 50  0000 C CNN
 F 1 "330" V 9200 4900 50  0000 C CNN
-F 2 "Resistors_SMD:R_0805_HandSoldering" V 9130 4900 50  0001 C CNN
+F 2 "Resistors_SMD:R_1206_HandSoldering" V 9130 4900 50  0001 C CNN
 F 3 "" H 9200 4900 50  0000 C CNN
 	1    9200 4900
@@
 F 0 "D3" H 9150 5275 50  0000 L CNN
 F 1 "Led_Small" H 9025 5050 50  0000 L CNN
-F 2 "LEDs:LED_0805" V 9200 5150 50  0001 C CNN
+F 2 "LEDs:LED_1206" V 9200 5150 50  0001 C CNN
 F 3 "" V 9200 5150 50  0000 C CNN
 	1    9200 5150
@@
 F 0 "R24" V 4980 3500 50  0000 C CNN
 F 1 "10k" V 4900 3500 50  0000 C CNN
-F 2 "Resistors_SMD:R_0805_HandSoldering" V 4830 3500 50  0001 C CNN
+F 2 "Resistors_SMD:R_1206_HandSoldering" V 4830 3500 50  0001 C CNN
 F 3 "" H 4900 3500 50  0000 C CNN
 	1    4900 3500
@@
 F 0 "R25" V 4980 3700 50  0000 C CNN
 F 1 "10k" V 4900 3700 50  0000 C CNN
-F 2 "Resistors_SMD:R_0805_HandSoldering" V 4830 3700 50  0001 C CNN
+F 2 "Resistors_SMD:R_1206_HandSoldering" V 4830 3700 50  0001 C CNN
 F 3 "" H 4900 3700 50  0000 C CNN
 	1    4900 3700
@@
 F 0 "R26" V 4980 3900 50  0000 C CNN
 F 1 "10k" V 4900 3900 50  0000 C CNN
-F 2 "Resistors_SMD:R_0805_HandSoldering" V 4830 3900 50  0001 C CNN
+F 2 "Resistors_SMD:R_1206_HandSoldering" V 4830 3900 50  0001 C CNN
 F 3 "" H 4900 3900 50  0000 C CNN
 	1    4900 3900
@@
 F 0 "R27" V 2380 6750 50  0000 C CNN
 F 1 "4.7k" V 2300 6750 50  0000 C CNN
-F 2 "Resistors_SMD:R_0805_HandSoldering" V 2230 6750 50  0001 C CNN
+F 2 "Resistors_SMD:R_1206_HandSoldering" V 2230 6750 50  0001 C CNN
 F 3 "" H 2300 6750 50  0000 C CNN
 	1    2300 6750
