File: hw/usbavrfloppy.sch (KiCad schematic (older format))
At the start: 63 parts, among them CON1 Conn_02x03, J1 bothdrv, J2 floppy_conn, J3 floppy_power, J4 FPC Floppy, J5 USB_B, J6 PWRIN, J7 USB_OTG, P1 CONN_01X03, P2 CONN_01X01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

Commit message: Updated
Changed lines of the file:
@@
 Sheet 1 1
 Title "USB AVR Amiga Floppy Controller"
-Date "2018-03-01"
-Rev "1"
+Date "2021-03-22"
+Rev "2"
 Comp "RetroBit Lab"
 Comment1 "Creative Commons Attribution Share-Alike (CC BY-SA)"
@@
 Text Label 4050 7150 2    60   ~ 0
 ~mSTEP
-Text Label 9350 2600 2    60   ~ 0
+Text Label 9350 2600 2    47   ~ 0
 ~TRK0
 Text Label 6400 1450 0    60   ~ 0
 ~TRK0
-Text Label 9350 2900 2    60   ~ 0
+Text Label 9350 2900 2    47   ~ 0
 ~SIDE1
 Text Label 8250 1450 0    60   ~ 0
 ~SIDE1
-Text Label 9350 2500 2    60   ~ 0
+Text Label 9350 2500 2    47   ~ 0
 ~WGATE
 Text Label 6400 2800 0    60   ~ 0
@@
 Text Label 8300 2800 0    60   ~ 0
 ~WPROT
-Text Label 9350 2700 2    60   ~ 0
+Text Label 9350 2700 2    47   ~ 0
 ~WPROT
-Text Label 9350 1700 2    60   ~ 0
+Text Label 9350 1700 2    47   ~ 0
 ~INDEX
 Wire Wire Line
@@
 Text Label 6400 4150 0    60   ~ 0
 ~INDEX
-Text Label 9350 2400 2    60   ~ 0
+Text Label 9350 2400 2    47   ~ 0
 ~WDATA
 Text Label 8200 4150 0    60   ~ 0
 ~WDATA
-Text Label 9350 2800 2    60   ~ 0
+Text Label 9350 2800 2    47   ~ 0
 ~RDATA
 Text Label 6400 5500 0    60   ~ 0
@@
 Text Label 6400 7150 0    60   ~ 0
 ~DIR
-Text Label 9350 2200 2    60   ~ 0
+Text Label 9350 2200 2    47   ~ 0
 ~DIR
 Text Label 4900 7150 0    60   ~ 0
 ~STEP
-Text Label 9350 2300 2    60   ~ 0
+Text Label 9350 2300 2    47   ~ 0
 ~STEP
 Text GLabel 2450 750  0    60   Input ~ 0
@@
 	10200 2550 10500 2550
 Wire Wire Line
-	10800 3350 10450 3350
-Wire Wire Line
-	10450 3350 10450 2650
-Wire Wire Line
 	10200 2650 10450 2650
 Wire Wire Line
@@
 Wire Wire Line
 	10300 3900 10800 3900
+Wire Wire Line
+	10450 2650 10450 3300
+Wire Wire Line
+	10450 3300 10800 3300
 $EndSCHEMATC

Commit message: Modified for final Kicad 5
Parts:
- CON1: footprint Connector_PinHeader_2.54mm:PinHeader_2x03_P2.54mm_Horizontal -> Connector_IDC:IDC-Header_2x03_P2.54mm_Vertical
Changed lines of the file:
@@
 F 0 "CON1" H 10350 5650 50  0000 C CNN
 F 1 "Conn_02x03" H 10250 5150 50  0000 C CNN
-F 2 "Connector_PinHeader_2.54mm:PinHeader_2x03_P2.54mm_Horizontal" H 10300 5400 50  0001 C CNN
+F 2 "Connector_IDC:IDC-Header_2x03_P2.54mm_Vertical" H 10300 5400 50  0001 C CNN
 F 3 "~" H 10300 5400 50  0001 C CNN
 	1    10300 5400
