File: hw/usbavrfloppy.kicad_pcb (KiCad board)
At the start: 2 copper layers, 96.5 x 70.5 mm, 65 parts, among them CON1 CONN_02X03, J1 bothdrv, J2 floppy_conn, J3 floppy_power, J5 USB_B, J6 PWRIN, J7 USB_OTG, P1 CONN_01X03, P2 CONN_01X01, P3 CONN_01X01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

Commit message: Changed backside (SilkScreen Back) logo and text
Parts:
- removed LOGO: LOGO, RetroBitLab:amigaLogo_BW_31x12mm-SilkScreenBack
- added G***: LOGO, RetroBitLab:amigaLogo_BW_31x12mm, B.Cu at (153.7, 100.3)
